File: KiCad/ESP32DUALDIAL.sch (KiCad schematic (older format))
At the start: 49 parts, among them J1 SERVICE, J2 100V IN, J3 FAN, J4 FAN, J5 POWER CONTROL, Q1 Q_NMOS_GDS, SW1 Rotary_Encoder_Switch, SW2 Rotary_Encoder_Switch, U1 CR2013-MI2120, U2 ESP-WROOM-32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

Commit message: change SSR SHARP S108T02
Parts:
- removed C4, C9: 10u, Capacitor_SMD:C_0402_1005Metric, symbol Device:C
- removed C5, C7: 0.1uF, Resistor_SMD:R_0603_1608Metric, symbol Device:C
- removed C8: 3900p, Capacitor_SMD:C_1206_3216Metric, symbol Device:C
- removed H5, H6: MountingHole_Pad, MountingHole:MountingHole_3.2mm_M3_Pad, symbol Mechanical:MountingHole_Pad
- removed J5: POWER CONTROL, TerminalBlock:TerminalBlock_bornier-5_P5.08mm, symbol Connector:Conn_01x05_Male
- removed L1: INDUCTOR, library:CD54PowerInductorSMD, symbol pspice:INDUCTOR
- removed R11: 10k, Resistor_SMD:R_0603_1608Metric, symbol Device:R
- removed R12: 100k, Resistor_SMD:R_0603_1608Metric, symbol Device:R
- removed R13: 6.8k, Resistor_SMD:R_0603_1608Metric, symbol Device:R
- removed U3: Mini-360, library:Mini-360_DCDC_LM2596_module, symbol Regulator_Linear:AMS1117CD-3.3
- removed U9: MP2307_DCDC_MPS, Package_SO:SOIC-8-1EP_3.9x4.9mm_P1.27mm_EP2.514x3.2mm, symbol nanbuwks:MP2307_DCDC_MPS
- added J5: Conn_01x02_Male, TerminalBlock:TerminalBlock_bornier-2_P5.08mm, symbol Connector:Conn_01x02_Male
- added J6: Conn_01x06_Male, TerminalBlock:TerminalBlock_bornier-6_P5.08mm, symbol Connector:Conn_01x06_Male
- added JP1: Jumper, Jumper:SolderJumper-2_P1.3mm_Bridged_Pad1.0x1.5mm, symbol Device:Jumper
- added JP2: Jumper_NC_Dual, Jumper:SolderJumper-3_P1.3mm_Bridged12_RoundedPad1.0x1.5mm_NumberLabels, symbol Device:Jumper_NC_Dual
- added U3: QS-1205CME-3A_MINIDC-DC_12-24Vto5V3A_1.8V_2.5V_3.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, library:QS-1205CME-3A_MINIDC-DC_12-24Vto5V3A_1.8V_2.5V_3.3V_5V_9V_12V, symbol nanbuwks:QS-1205CME-3A_MINIDC-DC_12-24Vto5V3A_1.8V_2.5V_3.3V_5V_9V_12V
- added U9: TBD62783A, Package_DIP:DIP-18_W7.62mm, symbol Transistor_Array:TBD62783A
- R4: value 26.1k -> NC
- R5, R6, R7, R8: value 220 -> 330
- U5, U6, U7, U8: value S112S01 -> S108T02; footprint library:SSR_NNC_NNG1D -> library:SSR_SHARP_S108T02
Connections:
- no-connect marks 17 -> 24
Other:
- note added: "PUMPA\nPUMPB\nOZON0A\nOZON0B\nOZON1A\nOZON1B\nOZON2A\nOZON2B"
- note removed: "COMMON\nPUMP\nOZON0\nOZON1\nOZON2"
- moved on the sheet: BZ1, C1, C2, C3, C6, F1, H1, H2, H3, H4, J1, J2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

Commit message: version 20210119
Parts:
- removed J2: 100V IN, TerminalBlock:TerminalBlock_bornier-2_P5.08mm, symbol Connector:Conn_01x02_Male
- removed J5: Conn_01x02_Male, TerminalBlock:TerminalBlock_bornier-2_P5.08mm, symbol Connector:Conn_01x02_Male
- removed J6: Conn_01x06_Male, TerminalBlock:TerminalBlock_bornier-6_P5.08mm, symbol Connector:Conn_01x06_Male
- added C10, C11: 10u, Capacitor_SMD:C_0402_1005Metric, symbol Device:C
- added C12, C4, C5, C7, C8, C9: 0.1uF, Resistor_SMD:R_0603_1608Metric, symbol Device:C
- added D1: D_Schottky, Diode_SMD:D_SOD-123F, symbol Device:D_Schottky
- added J2: Conn_01x04_Male, Connector_JST:JST_NV_B04P-NV_1x04_P5.00mm_Vertical, symbol Connector:Conn_01x04_Male
- added J5: Conn_01x03_Male, Connector_JST:JST_VH_B3P-VH_1x03_P3.96mm_Vertical, symbol Connector:Conn_01x03_Male
- added J6, J7, J8: Conn_01x02_Male, Connector_JST:JST_NV_B02P-NV_1x02_P5.00mm_Vertical, symbol Connector:Conn_01x02_Male
- F1: footprint Fuse:Fuse_Littelfuse-LVR200 -> library:20mmFuse_P5x2
Connections:
- net +12V: now also C11.2, D1.1 (K)
- net GND: now also C10.1, C12.2, C4.2, C5.2, C7.2, C8.2, C9.2
- net at SW1.A, U2.12 (IO27): now also C8.1
- net at SW1.B, U2.11 (IO26): now also C9.1
- net at SW1.S2, U2.10 (IO25): now also C4.1
- net at PS1.1 (AC/L), U5.2, U6.2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: now also F1.1
- net at F1.2: now also J2.2 (Pin_2)
- net at PS1.2 (AC/N): now also J2.1 (Pin_1), J5.3 (Pin_3), J6.2 (Pin_2), J7.2 (Pin_2), J8.2 (Pin_2); no longer F1.1
- net at SW2.S2, U2.13 (IO14): now also C12.1
- net at SW2.B, U2.14 (IO12): now also C7.1
- net at SW2.A, U2.16 (IO13): now also C5.1
- net at U5.1: now also J5.1 (Pin_1)
- net at U6.1: now also J6.1 (Pin_1)
- net at U7.1: now also J7.1 (Pin_1)
- net at U8.1: now also J8.1 (Pin_1)
- net at J3.2 (Pin_2), J4.2 (Pin_2), Q1.2 (D): now also C11.1, D1.2 (A)
- net at C6.1, Q1.1 (G), R10.2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: now also C10.2
- new net: J2.3 (Pin_3), J2.4 (Pin_4)
- no-connect marks 24 -> 25
Other:
- note added: "3.3V\nGND\n5V\nRX\nTX\n3.3V(WRITE)\nmode\nGND(RUN)\nRESET\nGND"
- note added: "AC/N\nHEAT FUSE\nHEAT FUSE\nAC/L"
- note added: "FAN OUTPUT"
- note added: "GPIO"
- note added: "PUMPA\n\nPUMPB\n"
- note added: "\nOZON0A\nOZON0B\n\nOZON1A\nOZON1B\n\nOZON2A\nOZON2B"
- note removed: "3.3V\nGND\n5V\nTX\nRX\n3.3V(WRITE)\nmode\nGND(RUN)\nRESET\nGND"
- note removed: "PUMPA\nPUMPB\nOZON0A\nOZON0B\nOZON1A\nOZON1B\nOZON2A\nOZON2B"
- moved on the sheet: C6, F1, J3, J4, R10, R9
