File: KiCad/ESP32DUALDIAL.kicad_pcb (KiCad board)
At the start: 2 copper layers, 180.5 x 74 mm, 82 parts, among them J1 SERVICE, J2 Conn_01x04_Male, J3 mode, J5 Conn_01x03_Male, J6 Conn_01x02_Male, J7 Conn_01x02_Male, J8 Conn_01x02_Male, M1 Fan_CPU_4pin, M2 Fan_CPU_4pin, Q1 Q_NMOS_GDS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

Commit message: change to V8.1
Parts:
- removed R19, R21: 10k, Resistor_SMD:R_0603_1608Metric
- moved TP8 68.1 mm to (162.7, 143.3)
- moved R22 25.6 mm to (179.3, 87.1), turned to -90 degrees
- moved R17 1.01 mm to (171.9, 87.1)
- moved R3 0.96 mm to (169.5, 87.1)
- moved R20 0.90 mm to (174.4, 87.1)
- moved R18 0.81 mm to (176.9, 87.1)
- turned U2 to -158 degrees
Routing:
- net Net-(D1-A): track 108.9 -> 38.7 mm, vias 2 -> 0
- net +3V3: track 278.2 -> 229.4 mm, vias 5 -> 3
- net Net-(U2-IO13): track 114.3 -> 98.1 mm, vias 2 -> 0
- net Net-(U2-IO12): track 121.8 -> 108.7 mm, vias 2 -> 0
- net +12V: track 199.3 -> 186.2 mm
- net OZON1: track 84.3 -> 79.5 mm, vias 0 -> 2
- net OZON0: track 71.6 -> 68.8 mm
- net Net-(U2-IO35): track 56.0 -> 53.5 mm
- net Net-(U2-IO15): track 101.9 -> 99.6 mm
- net OZON2: track 76.8 -> 74.6 mm
- net Net-(U2-IO0): track 40.7 -> 42.6 mm
- net BUZZER: track 72.1 -> 73.5 mm
- net RESET: track 41.1 -> 40.0 mm
- net Net-(J1-Pin_4): track 38.4 -> 39.4 mm
Other:
- board text added: "10k x 5"
- board text added: "270 -1k x 3"
- board text added: "270-1k x 7"
- board text added: "ESP-32 DUALDIAL V8.1"
- board text removed: "10k x 3"
- board text removed: "10k x 4"
- board text removed: "270 x 3"
- board text removed: "270-470 x 7"
- board text removed: "ESP-32 DUALDIAL V8"

Commit message: change to V8.2
Parts:
- added C15: 0.1uF, Capacitor_SMD:C_0603_1608Metric, F.Cu at (167.5, 93.6)
- added C16: 0.1uF, Capacitor_SMD:C_0603_1608Metric, F.Cu at (135.1, 98.3)
- added C17: 0.1uF, Capacitor_SMD:C_0603_1608Metric, F.Cu at (167.5, 96.6)
- added C18: 22uF, Capacitor_THT:CP_Radial_D6.3mm_P2.50mm, F.Cu at (169.9, 90.8)
- added C19: 220uF, Capacitor_THT:CP_Radial_D5.0mm_P2.00mm, F.Cu at (169.9, 97.0)
- moved C3 6.20 mm to (201.9, 104.7), turned to 90 degrees
- moved R3 3.90 mm to (173.1, 85.6)
- moved R17 3.71 mm to (175.3, 85.6)
- moved C2 3.05 mm to (203.7, 108.9), turned to -90 degrees
- moved R20 3.03 mm to (177.2, 85.9)
- moved R18 2.40 mm to (179.3, 86.9)
- moved R22 2.28 mm to (181.4, 88.0)
- moved C1 2.15 mm to (200.4, 100.5), turned to 90 degrees
- moved TP1 1.58 mm to (179.5, 91.0)
- moved TP2 1.58 mm to (182.5, 91.0)
- moved TP3 1.58 mm to (185.5, 91.0)
- moved R2 0.95 mm to (200.2, 97.4)
Routing:
- net Earth: track 211.1 -> 228.7 mm
- net +3V3: track 229.4 -> 240.6 mm
- net Net-(J1-Pin_7): track 18.3 -> 14.3 mm
- net BUZZER: track 73.5 -> 77.4 mm
- net Net-(U2-IO25): track 49.4 -> 45.6 mm
- net OZON1: track 79.5 -> 82.8 mm
- net OZON0: track 68.8 -> 66.2 mm
- net OZON2: track 74.6 -> 72.0 mm
- net Net-(U2-IO15): track 99.6 -> 102.0 mm
- net PUMP: track 63.2 -> 61.3 mm
- net Net-(U2-IO0): track 42.6 -> 44.4 mm
- net Net-(U2-IO14): track 127.6 -> 126.6 mm
- net Net-(U2-IO34): track 44.8 -> 45.6 mm
- net Net-(U2-IO12): track 108.7 -> 109.5 mm
- net Net-(U2-IO35): track 53.5 -> 54.1 mm
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Other:
- board text added: "ESP-32 DUALDIAL V8.2"
- board text removed: "ESP-32 DUALDIAL V8.1"
